File: Hardware/SparkFun_ENS160_BME280_Breakout.brd (EAGLE design)
At the start: 25.4 x 25.4 mm, 64 parts, among them J1 Qwiic Right Angle, J3 Qwiic Right Angle, J4 PTH, U1 AP2127K-1.8V, U2 ENS-160, U3 BME280

Commit message: added a 100nF cap to VDDIO on BME280
-added C6
-re-routed 3V3 and GND for better return path to GND pads on ICs
Parts:
- added C6: 0.1uF, SparkFun-Capacitors:0402-TIGHT
- moved R1 1.45 mm to (12.2, 8.99)
- moved C1 0.72 mm to (17.5, 15.8), turned to 90 degrees
Connections:
- removed net !INT: INT.1
- net !INT!: now also INT.1
- net 3.3V: now also C6.1
- net GND: now also C6.2
Routing:
- net !INT!: track 0.00 -> 17.6 mm
- net 3.3V: track 71.5 -> 79.3 mm, vias 8 -> 10
- net GND: track 1.74 -> 3.36 mm, vias 29 -> 42
- net N$3: track 2.55 -> 0.97 mm
- net SDO/ADR: track 6.33 -> 4.86 mm
- net SCL: track 42.0 -> 43.2 mm
- net SDA: track 33.8 -> 35.0 mm
- added copper zone on layer 16, net 3.3V
